Commit message: added target drone

File: gym_pybullet_drones/assets/custom.urdf (robot description, URDF)
Before this commit: robot cf2, 6 links, 5 joints
Links:
- link base_link: geometry collision cylinder length=.025 radius=.06; visual mesh filename=./drone_normal_zup.obj scale=0.001 0.001 0.001

Commit message: added RL env

File: gym_pybullet_drones/assets/custom.urdf (robot description, URDF)
Before this commit: robot cf2, 6 links, 5 joints
Links:
- link base_link: mass 0.027 -> 0.725977

Commit message: imu params fix and inertia

File: gym_pybullet_drones/assets/custom.urdf (robot description, URDF)
Before this commit: robot cf2, 6 links, 5 joints
Links:
- link base_link: geometry collision box size=.32 .35 .05; visual mesh filename=./drone_normal_zup.obj scale=0.001 0.001 0.001
